File: bbq_sensor.kicad_sch (KiCad schematic)
At the start: 3 parts, among them J1 Conn_01x06_Socket, P1 Connector_Generic:Conn_01x08, P2 Connector_Generic:Conn_01x08

Commit message: improved pcb
Parts:
- removed J1: Conn_01x06_Socket, Connector_PinHeader_2.54mm:PinHeader_1x06_P2.54mm_Vertical, symbol Connector:Conn_01x06_Socket
- removed P1, P2: Connector_Generic:Conn_01x08, D1_mini:D1_mini_Pin_Header, symbol Connector_Generic:Conn_01x08
- added J1: Conn_01x02_Socket, Connector_JST:JST_EH_B2B-EH-A_1x02_P2.50mm_Vertical, symbol Connector:Conn_01x02_Socket
- added M1: ~, tp4056-module:tp4056-module, symbol tp4056:tp4056
- added U1: LM1117DT-3.3, Package_TO_SOT_SMD:SOT-89-3_Handsoldering, symbol Regulator_Linear:LM1117DT-3.3
- added U2: WEMOS_D1_mini, RF_Module:WEMOS_D1_mini_light, symbol RF_Module:WEMOS_D1_mini
Other:
- note removed: "D1 Mini Shield"
- note removed: "GPIO0"
- note removed: "GPIO12"
- note removed: "GPIO13"
- note removed: "GPIO14"
- note removed: "GPIO15"
- note removed: "GPIO16"
- note removed: "GPIO2"
- note removed: "GPIO4"
- note removed: "GPIO5"

Commit message: update board
Parts:
- added J2: USB-C_Conn, Connector_JST:JST_EH_B2B-EH-A_1x02_P2.50mm_Vertical, symbol Connector:Conn_01x02_Socket
- added J3: Conn_01x06_Socket, Connector_PinSocket_2.54mm:PinSocket_1x06_P2.54mm_Vertical, symbol Connector:Conn_01x06_Socket
- J1: value Conn_01x02_Socket -> Battery_Conn
- U1: value LM1117DT-3.3 -> HT7333
Connections:
- net at U2.10 (GND): now also J3.4 (GND)
- net at U2.13 (SDA/D2): now also J3.2 (D2_CS)
- net at U2.14 (SCL/D1): now also J3.1 (D1_CLK)
- net at U2.3 (D0): now also J3.3 (D0_DO)
- net at U2.8 (3V3): now also U1.3 (VOUT)
- net at U2.9 (5V): now also J3.6 (VIN)
- net at U1.1 (VIN): now also M1.3 (Vout+)
- net at U1.2 (GND): now also M1.4 (Vout-)
- net at M1.1 (Vin+): now also J2.2 (Vin+)
- net at M1.2 (Vin-): now also J2.1 (Vin-)
- net at M1.5 (B+): now also J1.2 (Battery_+)
- net at M1.6 (B-): now also J1.1 (Battery_-)
Other:
- moved on the sheet: U1

Commit message: added caps
Parts:
- added C1, C5: 47 µF MLCC, Capacitor_SMD:C_1206_3216Metric_Pad1.33x1.80mm_HandSolder, symbol Device:C_Small_US
- added C2: 100 µF Elco, Capacitor_SMD:C_1206_3216Metric_Pad1.33x1.80mm_HandSolder, symbol Device:C_Small_US
- added C3: 10 µF MLCC, Capacitor_SMD:C_1206_3216Metric_Pad1.33x1.80mm_HandSolder, symbol Device:C_Small_US
- added C4, C6: 0.1 µF MLCC, Capacitor_SMD:C_1206_3216Metric_Pad1.33x1.80mm_HandSolder, symbol Device:C_Small_US
Connections:
- net at J3.4 (GND), U2.10 (GND): now also M1.4 (Vout-), U1.2 (GND), C1.2, C2.2, C3.2, C4.2, C5.2, C6.2
- net at U1.3 (VOUT), U2.8 (3V3): now also C3.1, C4.1, C5.1, C6.1
- net at M1.3 (Vout+), U1.1 (VIN): now also C1.1, C2.1
Other:
- moved on the sheet: J1, J2, J3, M1, U1, U2
