File: bbq_sensor.kicad_pcb (KiCad board)
At the start: 2 copper layers, 25.5 x 30 mm, 3 parts, among them J1 Conn_01x06_Socket, P1 Connector_Generic:Conn_01x08, P2 Connector_Generic:Conn_01x08

Commit message: improved pcb
Parts:
- removed P1, P2: Connector_Generic:Conn_01x08, D1_mini:D1_mini_Pin_Header
- added J1: Conn_01x02_Socket, Connector_JST:JST_EH_B2B-EH-A_1x02_P2.50mm_Vertical, F.Cu at (178.0, 105.5)
- added J2: Conn_01x02_Socket, Connector_JST:JST_EH_B2B-EH-A_1x02_P2.50mm_Vertical, F.Cu at (154.5, 106.0)
- added M1: ~, tp4056-module:tp4056-module, F.Cu at (149.0, 94.9)
- added U1: LM1117DT-3.3, Package_TO_SOT_SMD:SOT-89-3_Handsoldering, F.Cu at (167.0, 104.0)
- added U2: WEMOS_D1_mini, RF_Module:WEMOS_D1_mini_light, F.Cu at (177.9, 73.1)
- moved J1 12.4 mm to (142.0, 74.2), turned to 0 degrees
Routing:
- net /+3.3V: track 38.1 -> 0.00 mm, vias 1 -> 0
- net /GND: track 29.0 -> 0.00 mm
- net /D2: track 25.1 -> 0.00 mm, vias 1 -> 0
- net /D1: track 21.5 -> 0.00 mm
- net /D0: track 14.3 -> 0.00 mm
Other:
- board size 25.5 x 30 mm -> 79 x 79 mm
- board text removed: "3V3"
- board text removed: "5V"
- board text removed: "A0"
- board text removed: "D3"
- board text removed: "D4"
- board text removed: "D5"
- board text removed: "D6"
- board text removed: "D7"
- board text removed: "D8"
- board text removed: "G"
- board text removed: "RX"
- board text removed: "Rst"
- board text removed: "TX"

Commit message: update board
Parts:
- removed J1: Conn_01x06_Socket, Connector_PinHeader_2.54mm:PinHeader_1x06_P2.54mm_Vertical
- removed J1, J2: Conn_01x02_Socket, Connector_JST:JST_EH_B2B-EH-A_1x02_P2.50mm_Vertical
- added Battery: Battery_Conn, Connector_JST:JST_EH_B2B-EH-A_1x02_P2.50mm_Vertical, F.Cu at (157.3, 103.2)
- added MAX31855: MAX31855, Connector_PinSocket_2.54mm:PinSocket_1x06_P2.54mm_Vertical, F.Cu at (123.0, 74.3)
- added USB-C: USB-C_Conn, Connector_JST:JST_EH_B2B-EH-A_1x02_P2.50mm_Vertical, F.Cu at (177.0, 103.2)
- ESP8266 D1 Mini: renamed from U2
- HT7333: renamed from U1; value LM1117DT-3.3 -> HT7333
- moved HT7333 1.41 mm to (166.0, 105.0), turned to 180 degrees
- renumbered M1 to TP4056
Connections:
- ESP8266 D1 Mini pad 10: unconnected-(U2-GND-Pad10) -> Net-(J3-GND)
- ESP8266 D1 Mini pad 13: unconnected-(U2-SDA/D2-Pad13) -> Net-(J3-D2_CS)
- ESP8266 D1 Mini pad 14: unconnected-(U2-SCL/D1-Pad14) -> Net-(J3-D1_CLK)
- ESP8266 D1 Mini pad 3: unconnected-(U2-D0-Pad3) -> Net-(J3-D0_DO)
- ESP8266 D1 Mini pad 8: unconnected-(U2-3V3-Pad8) -> Net-(U1-VOUT)
- ESP8266 D1 Mini pad 9: unconnected-(U2-5V-Pad9) -> Net-(J3-VIN)
- HT7333 pad 1: unconnected-(U1-GND-Pad1) -> Net-(M1-Vout+)
- HT7333 pad 2: unconnected-(U1-VO-Pad2) -> Net-(M1-Vout-)
- HT7333 pad 3: unconnected-(U1-VI-Pad3) -> Net-(U1-VOUT)
- TP4056 pad 1: unconnected-(M1-Vin+-Pad1) -> Net-(J2-Vin+)
- TP4056 pad 2: unconnected-(M1-Vin--Pad2) -> Net-(J2-Vin-)
- TP4056 pad 3: unconnected-(M1-Vout+-Pad3) -> Net-(M1-Vout+)
- TP4056 pad 4: unconnected-(M1-Vout--Pad4) -> Net-(M1-Vout-)
- TP4056 pad 5: unconnected-(M1-B+-Pad5) -> Net-(J1-Battery_+)
- TP4056 pad 6: unconnected-(M1-B--Pad6) -> Net-(J1-Battery_-)
Routing:
- net Net-(J3-D1_CLK): track 0.00 -> 65.0 mm, vias 0 -> 1
- net Net-(J3-D2_CS): track 0.00 -> 58.9 mm
- net Net-(J3-D0_DO): track 0.00 -> 52.7 mm
- net Net-(M1-Vout-): track 0.00 -> 49.2 mm
- net Net-(M1-Vout+): track 0.00 -> 47.4 mm
- net Net-(J3-GND): track 0.00 -> 45.7 mm
- net Net-(J3-VIN): track 0.00 -> 40.8 mm
- net Net-(U1-VOUT): track 0.00 -> 38.4 mm, vias 0 -> 1
- net Net-(J1-Battery_-): track 0.00 -> 35.5 mm
- net Net-(J1-Battery_+): track 0.00 -> 34.7 mm
- net Net-(J2-Vin-): track 0.00 -> 33.9 mm
- net Net-(J2-Vin+): track 0.00 -> 33.8 mm

Commit message: added caps
Parts:
- added C1: 47 µF MLCC, Capacitor_SMD:C_1206_3216Metric_Pad1.33x1.80mm_HandSolder, F.Cu at (116.3, 105.6)
- added C2: 100 µF Elco, Capacitor_SMD:C_1206_3216Metric_Pad1.33x1.80mm_HandSolder, F.Cu at (116.5, 95.6)
- added C3: 10 µF MLCC, Capacitor_SMD:C_1206_3216Metric_Pad1.33x1.80mm_HandSolder, F.Cu at (163.3, 102.6)
- added C4: 0.1 µF MLCC, Capacitor_SMD:C_1206_3216Metric_Pad1.33x1.80mm_HandSolder, F.Cu at (167.5, 102.6)
- added C5: 47 µF MLCC, Capacitor_SMD:C_1206_3216Metric_Pad1.33x1.80mm_HandSolder, F.Cu at (162.0, 64.0)
- added C6: 0.1 µF MLCC, Capacitor_SMD:C_1206_3216Metric_Pad1.33x1.80mm_HandSolder, F.Cu at (162.0, 69.0)
- J3: renamed from MAX31855; value MAX31855 -> Conn_01x06_Socket
- U2: renamed from ESP8266 D1 Mini
- moved U1 6.02 mm to (163.8, 110.6)
- renumbered Battery to J1, USB-C to J2, TP4056 to M1, HT7333 to U1
Connections:
- M1 pad 4: Net-(M1-Vout-) -> Net-(J3-GND)
- U1 pad 1: Net-(M1-Vout+) -> Net-(J3-GND)
- U1 pad 2: Net-(M1-Vout-) -> Net-(M1-Vout+)
Routing:
- net Net-(J3-D1_CLK): track 65.0 -> 0.00 mm, vias 1 -> 0
- net Net-(J3-D2_CS): track 58.9 -> 0.00 mm
- net Net-(J3-D0_DO): track 52.7 -> 0.00 mm
- net Net-(M1-Vout-): track 49.2 -> 0.00 mm
- net Net-(M1-Vout+): track 47.4 -> 0.00 mm
- net Net-(J3-GND): track 45.7 -> 0.00 mm
- net Net-(J3-VIN): track 40.8 -> 0.00 mm
- net Net-(U1-VOUT): track 38.4 -> 0.00 mm, vias 1 -> 0
- net Net-(J1-Battery_-): track 35.5 -> 0.00 mm
- net Net-(J1-Battery_+): track 34.7 -> 0.00 mm
- net Net-(J2-Vin-): track 33.9 -> 0.00 mm
- net Net-(J2-Vin+): track 33.8 -> 0.00 mm

Commit message: update image
Parts:
- moved C2 8.91 mm to (116.1, 104.5)
- moved C1 8.61 mm to (115.9, 97.0)
- moved C5 0.40 mm to (162.0, 64.4)
- renumbered J1 to Battery, U1 to HT7333, J3 to MAX31855, M1 to TP4056, J2 to USB-C
Routing:
- net Net-(J3-GND): track 0.00 -> 132.5 mm, vias 0 -> 2
- net Net-(J3-D1_CLK): track 0.00 -> 65.5 mm, vias 0 -> 1
- net Net-(M1-Vout+): track 0.00 -> 65.0 mm
- net Net-(J3-D2_CS): track 0.00 -> 58.9 mm
- net Net-(U1-VOUT): track 0.00 -> 56.7 mm, vias 0 -> 2
- net Net-(J3-D0_DO): track 0.00 -> 52.8 mm
- net Net-(J3-VIN): track 0.00 -> 40.8 mm
- net Net-(J1-Battery_-): track 0.00 -> 35.5 mm
- net Net-(J1-Battery_+): track 0.00 -> 34.7 mm
- net Net-(J2-Vin+): track 0.00 -> 34.5 mm
- net Net-(J2-Vin-): track 0.00 -> 33.9 mm
